File: hardware/midi-solenoid-driver/midi-solenoid-driver.kicad_pcb (KiCad board)
At the start: 2 copper layers, 131.5 x 72 mm, 87 parts, among them J1 LEFT_DATA, J2 Conn_02x03_Odd_Even, J3 RIGHT_DATA, J4 12V_IN, J5 SOLENOIDS_OUT_1, J6 SOLENOIDS_OUT_2, Q1 Q_NMOS_GDS, Q10 Q_NMOS_GDS, Q11 Q_NMOS_GDS, Q12 Q_NMOS_GDS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

Commit message: Made v1.1 of driver board + gerbers
 - Added thermal relief to difficult-to-solder pads
 - Updated silkscreen
Other:
- board text added: "Willem Hillier rev1.1 19.222"
- board text removed: "Willem Hillier rev1 19.209"
Changed lines of the file:
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@@
     (mod_text_size 1 1)
     (mod_text_width 0.15)
-    (pad_size 4.600001 2.1)
-    (pad_drill 0)
+    (pad_size 2.78 2.78)
+    (pad_drill 1.78)
     (pad_to_mask_clearance 0.04572)
     (solder_mask_min_width 0.25)
@@
       (drillshape 0)
       (scaleselection 1)
-      (outputdirectory "gerbers/"))
+      (outputdirectory "gerbers-v1.1/"))
   )
   (net 0 "")
@@
     (descr "fuse holder, car blade fuse mini, http://www.keyelco.com/product-pdf.cfm?p=306")
     (tags "car blade fuse mini")
-    (zone_connect 2)
+    (zone_connect 1)
     (fp_text reference F1 (at 12.29 -2.795 180) (layer F.SilkS)
       (effects (font (size 1 1) (thickness 0.15)))
@@
     (fp_line (start -3.04 -1.67) (end -3.04 5.07) (layer F.Fab) (width 0.1))
     (pad 2 thru_hole circle (at 9.92 3.4 90) (size 2.78 2.78) (drill 1.78) (layers *.Cu *.Mask)
-      (net 3 +12V) (zone_connect 2))
+      (net 3 +12V) (zone_connect 1))
     (pad 2 thru_hole circle (at 9.92 0 90) (size 2.78 2.78) (drill 1.78) (layers *.Cu *.Mask)
-      (net 3 +12V) (zone_connect 2))
+      (net 3 +12V) (zone_connect 1))
     (pad 1 thru_hole circle (at 0 3.4 90) (size 2.78 2.78) (drill 1.78) (layers *.Cu *.Mask)
-      (net 5 /12V_FUSED1) (zone_connect 2))
+      (net 5 /12V_FUSED1) (zone_connect 1))
     (pad 1 thru_hole circle (at 0 0 90) (size 2.78 2.78) (drill 1.78) (layers *.Cu *.Mask)
-      (net 5 /12V_FUSED1) (zone_connect 2))
+      (net 5 /12V_FUSED1) (zone_connect 1))
     (model ${KISYS3DMOD}/Fuse.3dshapes/Fuseholder_Blade_Mini_Keystone_3568.wrl
       (at (xyz 0 0 0))
@@
     )
     (pad 1 thru_hole circle (at 0 0 90) (size 2.78 2.78) (drill 1.78) (layers *.Cu *.Mask)
-      (net 4 /12V_FUSED2) (zone_connect 2))
+      (net 4 /12V_FUSED2) (zone_connect 1))
     (pad 1 thru_hole circle (at 0 3.4 90) (size 2.78 2.78) (drill 1.78) (layers *.Cu *.Mask)
-      (net 4 /12V_FUSED2) (zone_connect 2))
+      (net 4 /12V_FUSED2) (zone_connect 1))
     (pad 2 thru_hole circle (at 9.92 0 90) (size 2.78 2.78) (drill 1.78) (layers *.Cu *.Mask)
-      (net 3 +12V) (zone_connect 2))
+      (net 3 +12V) (zone_connect 1))
     (pad 2 thru_hole circle (at 9.92 3.4 90) (size 2.78 2.78) (drill 1.78) (layers *.Cu *.Mask)
-      (net 3 +12V) (zone_connect 2))
+      (net 3 +12V) (zone_connect 1))
     (model ${KISYS3DMOD}/Fuse.3dshapes/Fuseholder_Blade_Mini_Keystone_3568.wrl
       (at (xyz 0 0 0))
@@
     (descr "terminal block Metz Connect Type701_RT11L02HGLU, 2 pins, pitch 6.35mm, size 12.7x12.5mm^2, drill diamater 1.3mm, pad diameter 2.5mm, see http://www.metz-connect.com/de/system/files/productfiles/Datenblatt_317011_RT11LxxHGLU_OFF-022798U.pdf, script-generated using https://github.com/pointhi/kicad-footprint-generator/scripts/TerminalBlock_MetzConnect")
     (tags "THT terminal block Metz Connect Type701_RT11L02HGLU pitch 6.35mm size 12.7x12.5mm^2 drill 1.3mm pad 2.5mm")
-    (zone_connect 2)
+    (zone_connect 1)
     (fp_text reference J4 (at 10.749 -3.839) (layer F.SilkS)
       (effects (font (size 1 1) (thickness 0.15)))
@@
     )
     (pad 1 thru_hole rect (at 0 0 180) (size 2.5 2.5) (drill 1.3) (layers *.Cu *.Mask)
-      (net 1 GND) (zone_connect 2))
+      (net 1 GND) (zone_connect 1))
     (pad 2 thru_hole circle (at 6.35 0 180) (size 2.5 2.5) (drill 1.3) (layers *.Cu *.Mask)
-      (net 3 +12V) (zone_connect 2))
+      (net 3 +12V) (zone_connect 1))
     (model ${KISYS3DMOD}/TerminalBlock_MetzConnect.3dshapes/TerminalBlock_MetzConnect_Type701_RT11L02HGLU_1x02_P6.35mm_Horizontal.wrl
       (at (xyz 0 0 0))
@@
     (effects (font (size 2.5 2.5) (thickness 0.3)) (justify left mirror))
   )
-  (gr_text "Willem Hillier rev1 19.209" (at 312.534 119.056) (layer B.SilkS)
+  (gr_text "Willem Hillier rev1.1 19.222" (at 312.534 119.056) (layer B.SilkS)
     (effects (font (size 1.25 1.25) (thickness 0.2)) (justify left mirror))
   )

Commit message: AddedRS485 transceiver, need to ship new rev
Parts:
- removed R1: 330R, Resistor_SMD:R_0603_1608Metric
- added C9: 0.1uF, Capacitor_SMD:C_0603_1608Metric, F.Cu at (308.6, 101.0)
- added U3: SN75LBC176D, Package_SO:SOIC-8_3.9x4.9mm_P1.27mm, F.Cu at (313.2, 105.3)
- SW2: value MIDI_NOTE_RANGE -> SW_DIP_x08
Connections:
- net Net-(J1-Pad4) renamed /RS485_B
- J1 pad 3: GND -> /RS485_A
- J3 pad 3: GND -> /RS485_A
- SW2 pad 1: /MIDI_NOTE_BIT6 -> /MIDI_NOTE_BIT0
- SW2 pad 15: (no net) -> GND
- SW2 pad 16: (no net) -> GND
- SW2 pad 2: /MIDI_NOTE_BIT5 -> /MIDI_NOTE_BIT1
- SW2 pad 3: /MIDI_NOTE_BIT4 -> /MIDI_NOTE_BIT2
- SW2 pad 5: /MIDI_NOTE_BIT2 -> /MIDI_NOTE_BIT4
- SW2 pad 6: /MIDI_NOTE_BIT1 -> /MIDI_NOTE_BIT5
- SW2 pad 7: /MIDI_NOTE_BIT0 -> /MIDI_NOTE_BIT6
Routing:
- net /RS485_A: track 0.00 -> 95.8 mm, vias 0 -> 2
- net /MIDI_NOTE_BIT0: track 24.3 -> 42.9 mm, vias 1 -> 2
- net /MIDI_IN: track 2.64 -> 18.7 mm, vias 0 -> 2
- net /MIDI_NOTE_BIT6: track 31.5 -> 17.8 mm
- net /RS485_B: track 114.4 -> 101.1 mm
- net /MIDI_NOTE_BIT1: track 24.5 -> 35.9 mm, vias 1 -> 2
- net /MIDI_NOTE_BIT5: track 29.7 -> 21.7 mm, vias 0 -> 2
- net /MIDI_NOTE_BIT2: track 26.3 -> 31.8 mm, vias 1 -> 2
- net /CTRL2: track 16.4 -> 20.6 mm
- net /MIDI_NOTE_BIT4: track 30.1 -> 26.3 mm, vias 1 -> 2
- net /CTRL1: track 17.4 -> 20.9 mm
- net +5V: track 86.8 -> 89.4 mm
- net /MIDI_NOTE_BIT3: track 28.2 -> 28.9 mm
- net GND: vias 125 -> 119
Other:
- board text added: "Willem Hillier rev1.2 19.226"
- board text removed: "Willem Hillier rev1.1 19.222"
