File: hardware/usb-serial-interface/usb-serial-interface.kicad_pcb (KiCad board)
At the start: 2 copper layers, 49.9 x 33 mm, 19 parts, among them J1 USB_B, J2 RJ12, U1 CP2102N-A01-GQFN24

Commit message: new usb serial gerbers
Parts:
- moved REF** 1.57 mm to (85.1, 80.3)
Changed lines of the file:
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@@
-(kicad_pcb (version 20171130) (host pcbnew 5.1.4-e60b266~84~ubuntu16.04.1)
+(kicad_pcb (version 20171130) (host pcbnew "(5.1.2)-2")
   (general
     (thickness 1.6)
@@
   )
   (module Symbol:OSHW-Logo2_9.8x8mm_SilkScreen (layer B.Cu)
-    (at 85.09 81.915 180)
+    (at 85.09 80.342 180)
     (descr "Open Source Hardware Symbol")
     (tags "Logo Symbol OSHW")
